File: KiCAD/STM32_Compute_Module.Rev1.0.kicad_sch (KiCad schematic)
At the start: 96 parts, among them J1 12V IN, J10 S6, J11 S7, J12 S8, J13 S9, J14 S10, J15 S11, J16 S12, J17 S13, J18 S14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

Commit message: Added manufacturing files and renamed
Connections:
- net +3.3V: no longer J34.1
- net +12V renamed VCC
- net VCC: now also J34.1
Other:
- title: STM32 Simple -> STM32_Compute_Module
