File: KiCAD/STM32_Compute_Module.Rev1.0.kicad_pcb (KiCad board)
At the start: 4 copper layers, 30 x 51 mm, 96 parts, among them J1 12V IN, J10 S6, J11 S7, J12 S8, J13 S9, J14 S10, J15 S11, J16 S12, J17 S13, J18 S14, J19 S15, J2 GND, J20 S16, J21 S17, J22 S18, J23 S19, J24 S20, J25 S21, J26 S22, J27 S23, J28 S24, J29 S25, J3 Tag Connect, J30 S26, J31 S27, J32 S28, J33 S29, J34 S30, J35 S31, J36 S32, J37 S33, J38 S34, J39 S35, J4 S1, J40 S36, J41 S37, J42 S38, J43 S39, J44 S40, J45 S41, J46 S42, J5 S2, J6 S3, J7 S4, J8 USB_C_Receptacle_USB2.0, J9 S5, Q1 AO3401A, SW1 SW_SPDT, SW2 SW_Push, SW3 SW_Push, SW4 SW_Push, U1 STM32F405RGT6, U3 USBLC6-2SC6, Y1 16MHz

Commit message: Added manufacturing files and renamed
Parts:
- added G***: LOGO, LOGO, B.Cu at (210.0, 83.4)
Connections:
- J1 pad 1: +12V -> VCC
- J34 pad 1: +3.3V -> VCC
- Q1 pad 3: +12V -> VCC
Routing:
- net VCC: track 0.00 -> 50.4 mm, vias 0 -> 2
- net +12V: track 4.70 -> 0.00 mm
- net +3.3V: track 42.2 -> 40.5 mm, vias 16 -> 15
- net +5V: track 66.5 -> 65.8 mm
Other:
- board text added: "06/2023"
- board text added: "STM32_DEV REV_1.0 5V-12V IN"
- board text added: "VCC"
- board text removed: "05/2023"
- board text removed: "12V"
- board text removed: "STM32_DEV REV_1.0"

Commit message: Added JLC PCB serial number location
Other:
- board text added: "JLCJLCJLCJLC"
Changed lines of the file:
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@@
     (effects (font (size 1 1) (thickness 0.16)) (justify right mirror))
+  )
+  (gr_text "JLCJLCJLCJLC" (at 186.4 87.2 -90) (layer "B.SilkS")
+    (effects (font (size 0.9 0.9) (thickness 0.15)) (justify left top mirror))
   )
   (gr_text "  29  " (at 215.4 106) (layer "B.SilkS")
